Commit message: First display of redblade on gazebo

File: redblade_description/urdf/redblade.xacro (robot description, xacro)
@@ -19,5 +19,5 @@
     <visual>
       <geometry>
-	<cylinder length="0.001" radius="0.01"/>
+  	<cylinder length="0.001" radius="0.01"/>
       </geometry>
       <material name="black"/>
@@ -32,9 +32,15 @@
     <visual>
       <geometry>
-	<box size="0.025 0.35 0.025"/>
+  	<box size="0.025 0.35 0.025"/>
       </geometry>
       <material name="grey"/>
       <origin rpy="0 0 0" xyz="0 0 0"/>
     </visual>
+    <collision>
+      <origin rpy="0 0 0" xyz="0 0 0"/>
+      <geometry>
+        <cylinder length="0.4" radius="3"/>
+      </geometry>
+    </collision>
     <inertial>
       <origin rpy="0 0 0" xyz="0 0 0"/>
@@ -48,36 +54,16 @@
     <origin xyz="0 0 0.195"/>
   </joint>
-  <!--	<link name="base_footprint">
-      <visual>
-      <geometry>
-      <cylinder length="0.001" radius="0.01"/>
-      </geometry>
-      <material name="black"/>
-      <origin rpy="0 0 0" xyz="0 0 0"/>
-      </visual>
-      <inertial>
-	<origin rpy="0 0 0" xyz="0 0 0"/>
-	<mass value="1"/>
-	<inertia ixx="0" ixy="0" ixz="0" iyy="0" iyz="0" izz="0"/>
-      </inertial>
-    </link>
-    <joint name="to_base_footprint" type="fixed">
-      <parent link="base_link"/>
-      <child link="base_footprint"/>
-      <origin xyz="0 0 -0.195"/>
-    </joint>
-    -->
     <link name="wheel_left">
       <visual>
-	<geometry>
-	  <cylinder length="0.12" radius="0.1975"/>
-	</geometry>
-	<material name="wheel"/>
-	<origin rpy="1.5707 0 0" xyz="0 0 0"/>
-      </visual>
-      <inertial>
-	<origin rpy="0 0 0" xyz="0 0 0"/>
-	<mass value="1"/>
-	<inertia ixx="1" ixy="0" ixz="0" iyy="1" iyz="0" izz="1"/>
+  	<geometry>
+  	  <cylinder length="0.12" radius="0.1975"/>
+  	</geometry>
+  	<material name="wheel"/>
+  	<origin rpy="1.5707 0 0" xyz="0 0 0"/>
+      </visual>
+      <inertial>
+  	<origin rpy="0 0 0" xyz="0 0 0"/>
+  	<mass value="1"/>
+  	<inertia ixx="1" ixy="0" ixz="0" iyy="1" iyz="0" izz="1"/>
       </inertial>
     </link>
@@ -89,14 +75,14 @@
     <link name="wheel_right">
       <visual>
-	<geometry>
-	  <cylinder length="0.12" radius="0.1975"/>
-	</geometry>
-	<material name="wheel"/>
-	<origin rpy="1.5707 0 0" xyz="0 0 0"/>
-      </visual>
-      <inertial>
-	<origin rpy="0 0 0" xyz="0 0 0"/>
-	<mass value="1"/>
-	<inertia ixx="1" ixy="0" ixz="0" iyy="1" iyz="0" izz="1"/>
+  	<geometry>
+  	  <cylinder length="0.12" radius="0.1975"/>
+  	</geometry>
+  	<material name="wheel"/>
+  	<origin rpy="1.5707 0 0" xyz="0 0 0"/>
+      </visual>
+      <inertial>
+  	<origin rpy="0 0 0" xyz="0 0 0"/>
+  	<mass value="1"/>
+  	<inertia ixx="1" ixy="0" ixz="0" iyy="1" iyz="0" izz="1"/>
       </inertial>
     </link>
@@ -108,14 +94,14 @@
     <link name="motor_mount_left">
       <visual>
-	<geometry>
-	  <box size="0.025 0.025 0.0575"/>
-	</geometry>
-	<material name="grey"/>
-	<origin rpy="0 0 0" xyz="0 0 0"/>
-      </visual>
-      <inertial>
-	<origin rpy="0 0 0" xyz="0 0 0"/>
-	<mass value="1"/>
-	<inertia ixx="1" ixy="0" ixz="0" iyy="1" iyz="0" izz="1"/>
+  	<geometry>
+  	  <box size="0.025 0.025 0.0575"/>
+  	</geometry>
+  	<material name="grey"/>
+  	<origin rpy="0 0 0" xyz="0 0 0"/>
+      </visual>
+      <inertial>
+  	<origin rpy="0 0 0" xyz="0 0 0"/>
+  	<mass value="1"/>
+  	<inertia ixx="1" ixy="0" ixz="0" iyy="1" iyz="0" izz="1"/>
       </inertial>
     </link>
@@ -127,14 +113,14 @@
     <link name="motor_mount_right">
       <visual>
-	<geometry>
-	  <box size="0.025 0.025 0.0575"/>
-	</geometry>
-	<material name="grey"/>
-	<origin rpy="0 0 0" xyz="0 0 0"/>
-      </visual>
-      <inertial>
-	<origin rpy="0 0 0" xyz="0 0 0"/>
-	<mass value="1"/>
-	<inertia ixx="1" ixy="0" ixz="0" iyy="1" iyz="0" izz="1"/>
+  	<geometry>
+  	  <box size="0.025 0.025 0.0575"/>
+  	</geometry>
+  	<material name="grey"/>
+  	<origin rpy="0 0 0" xyz="0 0 0"/>
+      </visual>
+      <inertial>
+  	<origin rpy="0 0 0" xyz="0 0 0"/>
+  	<mass value="1"/>
+  	<inertia ixx="1" ixy="0" ixz="0" iyy="1" iyz="0" izz="1"/>
       </inertial>
     </link>
@@ -146,14 +132,14 @@
     <link name="motor_area_bottom_left">
       <visual>
-	<geometry>
-	  <box size="0.585 0.025 0.025"/>
-	</geometry>
-	<material name="grey"/>
-	<origin rpy="0 0 0" xyz="0 0 0"/>
-      </visual>
-      <inertial>
-	<origin rpy="0 0 0" xyz="0 0 0"/>
-	<mass value="1"/>
-	<inertia ixx="1" ixy="0" ixz="0" iyy="1" iyz="0" izz="1"/>
+  	<geometry>
+  	  <box size="0.585 0.025 0.025"/>
+  	</geometry>
+  	<material name="grey"/>
+  	<origin rpy="0 0 0" xyz="0 0 0"/>
+      </visual>
+      <inertial>
+  	<origin rpy="0 0 0" xyz="0 0 0"/>
+  	<mass value="1"/>
+  	<inertia ixx="1" ixy="0" ixz="0" iyy="1" iyz="0" izz="1"/>
       </inertial>
     </link>
@@ -165,14 +151,14 @@
     <link name="motor_area_bottom_right">
       <visual>
-	<geometry>
-	  <box size="0.585 0.025 0.025"/>
-	</geometry>
-	<material name="grey"/>
-	<origin rpy="0 0 0" xyz="0 0 0"/>
-      </visual>
-      <inertial>
-	<origin rpy="0 0 0" xyz="0 0 0"/>
-	<mass value="1"/>
-	<inertia ixx="1" ixy="0" ixz="0" iyy="1" iyz="0" izz="1"/>
+  	<geometry>
+  	  <box size="0.585 0.025 0.025"/>
+  	</geometry>
+  	<material name="grey"/>
+  	<origin rpy="0 0 0" xyz="0 0 0"/>
+      </visual>
+      <inertial>
+  	<origin rpy="0 0 0" xyz="0 0 0"/>
+  	<mass value="1"/>
+  	<inertia ixx="1" ixy="0" ixz="0" iyy="1" iyz="0" izz="1"/>
       </inertial>
     </link>
@@ -184,14 +170,14 @@
     <link name="motor_area_bottom_front">
       <visual>
-	<geometry>
-	  <box size="0.025 0.255 0.025"/>
-	</geometry>
-	<material name="grey"/>
-	<origin rpy="0 0 0" xyz="0 0 0"/>
-      </visual>
-      <inertial>
-	<origin rpy="0 0 0" xyz="0 0 0"/>
-	<mass value="1"/>
-	<inertia ixx="1" ixy="0" ixz="0" iyy="1" iyz="0" izz="1"/>
+  	<geometry>
+  	  <box size="0.025 0.255 0.025"/>
+  	</geometry>
+  	<material name="grey"/>
+  	<origin rpy="0 0 0" xyz="0 0 0"/>
+      </visual>
+      <inertial>
+  	<origin rpy="0 0 0" xyz="0 0 0"/>
+  	<mass value="1"/>
+  	<inertia ixx="1" ixy="0" ixz="0" iyy="1" iyz="0" izz="1"/>
       </inertial>
     </link>
@@ -203,14 +189,14 @@
     <link name="motor_area_bottom_back">
       <visual>
-	<geometry>
-	  <box size="0.025 0.255 0.025"/>
-	</geometry>
-	<material name="grey"/>
-	<origin rpy="0 0 0" xyz="0 0 0"/>
-      </visual>
-      <inertial>
-	<origin rpy="0 0 0" xyz="0 0 0"/>
-	<mass value="1"/>
-	<inertia ixx="1" ixy="0" ixz="0" iyy="1" iyz="0" izz="1"/>
+  	<geometry>
+  	  <box size="0.025 0.255 0.025"/>
+  	</geometry>
+  	<material name="grey"/>
+  	<origin rpy="0 0 0" xyz="0 0 0"/>
+      </visual>
+      <inertial>
+  	<origin rpy="0 0 0" xyz="0 0 0"/>
+  	<mass value="1"/>
+  	<inertia ixx="1" ixy="0" ixz="0" iyy="1" iyz="0" izz="1"/>
       </inertial>
     </link>
@@ -222,14 +208,14 @@
     <link name="motor_area_vent_front_left">
       <visual>
-	<geometry>
-	  <box size="0.025 0.025 0.285"/>
-	</geometry>
-	<material name="grey"/>
-	<origin rpy="0 0 0" xyz="0 0 0"/>
-      </visual>
-      <inertial>
-	<origin rpy="0 0 0" xyz="0 0 0"/>
-	<mass value="1"/>
-	<inertia ixx="1" ixy="0" ixz="0" iyy="1" iyz="0" izz="1"/>
+  	<geometry>
+  	  <box size="0.025 0.025 0.285"/>
+  	</geometry>
+  	<material name="grey"/>
+  	<origin rpy="0 0 0" xyz="0 0 0"/>
+      </visual>
+      <inertial>
+  	<origin rpy="0 0 0" xyz="0 0 0"/>
+  	<mass value="1"/>
+  	<inertia ixx="1" ixy="0" ixz="0" iyy="1" iyz="0" izz="1"/>
       </inertial>
     </link>
@@ -241,14 +227,14 @@
     <link name="motor_area_vent_back_left">
       <visual>
-	<geometry>
-	  <box size="0.025 0.025 0.285"/>
-	</geometry>
-	<material name="grey"/>
-	<origin rpy="0 0 0" xyz="0 0 0"/>
-      </visual>
-      <inertial>
-	<origin rpy="0 0 0" xyz="0 0 0"/>
-	<mass value="1"/>
-	<inertia ixx="1" ixy="0" ixz="0" iyy="1" iyz="0" izz="1"/>
+  	<geometry>
+  	  <box size="0.025 0.025 0.285"/>
+  	</geometry>
+  	<material name="grey"/>
+  	<origin rpy="0 0 0" xyz="0 0 0"/>
+      </visual>
+      <inertial>
+  	<origin rpy="0 0 0" xyz="0 0 0"/>
+  	<mass value="1"/>
+  	<inertia ixx="1" ixy="0" ixz="0" iyy="1" iyz="0" izz="1"/>
       </inertial>
     </link>
@@ -260,14 +246,14 @@
     <link name="motor_area_vent_front_right">
       <visual>
-	<geometry>
-	  <box size="0.025 0.025 0.285"/>
-	</geometry>
-	<material name="grey"/>
-	<origin rpy="0 0 0" xyz="0 0 0"/>
-      </visual>
-      <inertial>
-	<origin rpy="0 0 0" xyz="0 0 0"/>
-	<mass value="1"/>
-	<inertia ixx="1" ixy="0" ixz="0" iyy="1" iyz="0" izz="1"/>
+  	<geometry>
+  	  <box size="0.025 0.025 0.285"/>
+  	</geometry>
+  	<material name="grey"/>
+  	<origin rpy="0 0 0" xyz="0 0 0"/>
+      </visual>
+      <inertial>
+  	<origin rpy="0 0 0" xyz="0 0 0"/>
+  	<mass value="1"/>
+  	<inertia ixx="1" ixy="0" ixz="0" iyy="1" iyz="0" izz="1"/>
       </inertial>
     </link>
@@ -279,14 +265,14 @@
     <link name="motor_area_vent_back_right">
       <visual>
-	<geometry>
-	  <box size="0.025 0.025 0.285"/>
-	</geometry>
-	w			<material name="grey"/>
-	<origin rpy="0 0 0" xyz="0 0 0"/>
-      </visual>
-      <inertial>
-	<origin rpy="0 0 0" xyz="0 0 0"/>
-	<mass value="1"/>
-	<inertia ixx="1" ixy="0" ixz="0" iyy="1" iyz="0" izz="1"/>
+  	<geometry>
+  	  <box size="0.025 0.025 0.285"/>
+  	</geometry>
+  	w			<material name="grey"/>
+  	<origin rpy="0 0 0" xyz="0 0 0"/>
+      </visual>
+      <inertial>
+  	<origin rpy="0 0 0" xyz="0 0 0"/>
+  	<mass value="1"/>
+  	<inertia ixx="1" ixy="0" ixz="0" iyy="1" iyz="0" izz="1"/>
       </inertial>
     </link>
@@ -298,14 +284,14 @@
     <link name="main_area_bottom_back">
       <visual>
-	<geometry>
-	  <box size="0.025 0.56 0.025"/>
-	</geometry>
-	<material name="grey"/>
-	<origin rpy="0 0 0" xyz="0 0 0"/>
-      </visual>
-      <inertial>
-	<origin rpy="0 0 0" xyz="0 0 0"/>
-	<mass value="1"/>
-	<inertia ixx="1" ixy="0" ixz="0" iyy="1" iyz="0" izz="1"/>
+  	<geometry>
+  	  <box size="0.025 0.56 0.025"/>
+  	</geometry>
+  	<material name="grey"/>
+  	<origin rpy="0 0 0" xyz="0 0 0"/>
+      </visual>
+      <inertial>
+  	<origin rpy="0 0 0" xyz="0 0 0"/>
+  	<mass value="1"/>
+  	<inertia ixx="1" ixy="0" ixz="0" iyy="1" iyz="0" izz="1"/>
       </inertial>
     </link>
@@ -317,14 +303,14 @@
     <link name="main_area_bottom_left">
       <visual>
-	<geometry>
-	  <box size="1.22 0.025 0.025"/>
-	</geometry>
-	<material name="grey"/>
-	<origin rpy="0 0 0" xyz="0 0 0"/>
-      </visual>
-      <inertial>
-	<origin rpy="0 0 0" xyz="0 0 0"/>
-	<mass value="1"/>
-	<inertia ixx="1" ixy="0" ixz="0" iyy="1" iyz="0" izz="1"/>
+  	<geometry>
+  	  <box size="1.22 0.025 0.025"/>
+  	</geometry>
+  	<material name="grey"/>
+  	<origin rpy="0 0 0" xyz="0 0 0"/>
+      </visual>
+      <inertial>
+  	<origin rpy="0 0 0" xyz="0 0 0"/>
+  	<mass value="1"/>
+  	<inertia ixx="1" ixy="0" ixz="0" iyy="1" iyz="0" izz="1"/>
       </inertial>
     </link>
@@ -336,14 +322,14 @@
     <link name="main_area_bottom_right">
       <visual>
-	<geometry>
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