Commit message: Added more control features

File: src/redblade_description/urdf/redblade.xacro (robot description, xacro)
@@ -10,4 +10,10 @@
   <xacro:property name="camera_link" value="0.05" /> <!-- Size of square 'camera' box -->
   <xacro:property name="axel_offset" value="0.05" /> <!-- Space btw top of beam and the each joint -->
+  <xacro:property name="base_wheel_width" value="0.12" />
+  <xacro:property name="base_wheel_radius" value="0.12" />
+  <xacro:property name="base_wheel_mass" value="1.0" />
+  <xacro:property name="caster_wheel_width" value="0.05" />
+  <xacro:property name="caster_wheel_radius" value="0.075" />
+  <xacro:property name="caster_wheel_mass" value="1.0" />
   <!-- Import all Gazebo-customization elements, including Gazebo colors -->
   <xacro:include filename="$(find redblade_description)/urdf/redblade.gazebo" />
@@ -37,10 +43,10 @@
       <origin rpy="0 0 0" xyz="0 0 0"/>
     </visual>
-    <collision>
-      <origin rpy="0 0 0" xyz="0 0 0"/>
-      <geometry>
-        <cylinder length="0.4" radius="3"/>
-      </geometry>
-    </collision>
+    <!-- <collision> -->
+    <!--   <origin rpy="0 0 0" xyz="0 0 0"/> -->
+    <!--   <geometry> -->
+    <!--     <cylinder length="0.4" radius="3"/> -->
+    <!--   </geometry> -->
+    <!-- </collision> -->
     <inertial>
       <origin rpy="0 0 0" xyz="0 0 0"/>
@@ -64,11 +70,22 @@
       <inertial>
   	<origin rpy="0 0 0" xyz="0 0 0"/>
-  	<mass value="1"/>
-  	<inertia ixx="1" ixy="0" ixz="0" iyy="1" iyz="0" izz="1"/>
-      </inertial>
+  	<mass value="${base_wheel_mass}"/>
+	<inertia ixx="1" ixy="0" ixz="0" iyy="1" iyz="0" izz="1"/>
+	<!-- <inertia ixx="${base_wheel_mass*base_wheel_radius*base_wheel_radius/4+base_wheel_mass*base_wheel_height*base_wheel_height)}"   -->
+	<!-- 	 ixy="0" ixz="0"  -->
+	<!-- 	 iyy="${base_wheel_mass*base_wheel_radius*base_wheel_radius/4+base_wheel_mass*base_wheel_height*base_wheel_height)}"   -->
+	<!-- 	 iyz="0" izz="${base_wheel_mass*base_wheel_radius*base_wheel_radius/2)}" /> -->
+      </inertial>
+    <collision>
+      <origin rpy="1.5707 0 0" xyz="0 0 0"/>
+      <geometry>
+        <cylinder length="0.12" radius="0.1975"/>
+      </geometry>
+    </collision>
     </link>
     <joint name="to_wheel_left" type="continuous">
       <parent link="base_link"/>
       <child link="wheel_left"/>
+      <axis xyz="0 1 0"/>
       <origin xyz="0 0.235 0"/>
     </joint>
@@ -86,8 +103,15 @@
   	<inertia ixx="1" ixy="0" ixz="0" iyy="1" iyz="0" izz="1"/>
       </inertial>
+      <collision>
+	<origin rpy="1.5707 0 0" xyz="0 0 0"/>
+	<geometry>
+	  <cylinder length="0.12" radius="0.1975"/>
+	</geometry>
+      </collision>
     </link>
     <joint name="to_wheel_right" type="continuous">
       <parent link="base_link"/>
       <child link="wheel_right"/>
+      <axis xyz="0 1 0"/>
       <origin xyz="0 -0.235 0"/>
     </joint>
@@ -1000,6 +1024,12 @@
   	<inertia ixx="1" ixy="0" ixz="0" iyy="1" iyz="0" izz="1"/>
       </inertial>
-    </link>
-    <joint name="to_caster_left" type="fixed">
+      <collision>
+	<origin rpy="1.5707 0 0" xyz="0 0 0"/>
+	<geometry>
+	  <cylinder length="0.05" radius="0.075"/>
+	</geometry>
+      </collision>
+    </link>
+    <joint name="to_caster_left" type="continuous">
       <parent link="deck_area_bottom_left"/>
       <child link="caster_left"/>
@@ -1019,6 +1049,12 @@
   	<inertia ixx="1" ixy="0" ixz="0" iyy="1" iyz="0" izz="1"/>
       </inertial>
-    </link>
-    <joint name="to_caster_right" type="fixed">
+      <collision>
+	<origin rpy="1.5707 0 0" xyz="0 0 0"/>
+	<geometry>
+	  <cylinder length="0.05" radius="0.075"/>
+	</geometry>
+      </collision>
+    </link>
+    <joint name="to_caster_right" type="continuous">
       <parent link="deck_area_bottom_right"/>
       <child link="caster_right"/>
@@ -1196,3 +1232,19 @@
       <origin rpy="0 0 0" xyz="0 0 0.87"/>
     </joint>
+  <transmission name="wheel_left_tran">
+    <type>transmission_interface/SimpleTransmission</type>
+    <joint name="to_wheel_left"/>
+    <actuator name="motor1">
+      <hardwareInterface>EffortJointInterface</hardwareInterface>
+      <mechanicalReduction>1</mechanicalReduction>
+    </actuator>
+  </transmission>
+  <transmission name="wheel_right_tran">
+    <type>transmission_interface/SimpleTransmission</type>
+    <joint name="to_wheel_right"/>
+    <actuator name="motor2">
+      <hardwareInterface>EffortJointInterface</hardwareInterface>
+      <mechanicalReduction>1</mechanicalReduction>
+    </actuator>
+  </transmission>
 </robot>

Commit message: Added more friction elements

File: src/redblade_description/urdf/redblade.xacro (robot description, xacro)
@@ -29,9 +29,4 @@
       <material name="black"/>
     </visual>
-    <inertial>
-      <origin rpy="0 0 0" xyz="0 0 0"/>
-      <mass value="1"/>
-      <inertia ixx="1" ixy="0" ixz="0" iyy="1" iyz="0" izz="1"/>
-    </inertial>
   </link>
   <link name="base_link">
@@ -43,10 +38,4 @@
       <origin rpy="0 0 0" xyz="0 0 0"/>
     </visual>
-    <!-- <collision> -->
-    <!--   <origin rpy="0 0 0" xyz="0 0 0"/> -->
-    <!--   <geometry> -->
-    <!--     <cylinder length="0.4" radius="3"/> -->
-    <!--   </geometry> -->
-    <!-- </collision> -->
     <inertial>
       <origin rpy="0 0 0" xyz="0 0 0"/>

Commit message: Modified inertia matrix

File: src/redblade_description/urdf/redblade.xacro (robot description, xacro)
@@ -16,4 +16,5 @@
   <xacro:property name="caster_wheel_radius" value="0.075" />
   <xacro:property name="caster_wheel_mass" value="1.0" />
+  <xacro:property name="torque" value="20.0" />
   <!-- Import all Gazebo-customization elements, including Gazebo colors -->
   <xacro:include filename="$(find redblade_description)/urdf/redblade.gazebo" />
@@ -60,9 +61,9 @@
   	<origin rpy="0 0 0" xyz="0 0 0"/>
   	<mass value="${base_wheel_mass}"/>
-	<inertia ixx="1" ixy="0" ixz="0" iyy="1" iyz="0" izz="1"/>
-	<!-- <inertia ixx="${base_wheel_mass*base_wheel_radius*base_wheel_radius/4+base_wheel_mass*base_wheel_height*base_wheel_height)}"   -->
-	<!-- 	 ixy="0" ixz="0"  -->
-	<!-- 	 iyy="${base_wheel_mass*base_wheel_radius*base_wheel_radius/4+base_wheel_mass*base_wheel_height*base_wheel_height)}"   -->
-	<!-- 	 iyz="0" izz="${base_wheel_mass*base_wheel_radius*base_wheel_radius/2)}" /> -->
+	<!-- <inertia ixx="1" ixy="0" ixz="0" iyy="1" iyz="0" izz="1"/> -->
+	<inertia ixx="${base_wheel_mass*base_wheel_radius*base_wheel_radius/4+base_wheel_mass*base_wheel_width*base_wheel_width)}"
+		 ixy="0" ixz="0"
+		 iyy="${base_wheel_mass*base_wheel_radius*base_wheel_radius/4+base_wheel_mass*base_wheel_width*base_wheel_width)}"
+		 iyz="0" izz="${base_wheel_mass*base_wheel_radius*base_wheel_radius/2)}" />
       </inertial>
     <collision>
@@ -89,6 +90,10 @@
       <inertial>
   	<origin rpy="0 0 0" xyz="0 0 0"/>
-  	<mass value="1"/>
-  	<inertia ixx="1" ixy="0" ixz="0" iyy="1" iyz="0" izz="1"/>
+   	<mass value="${base_wheel_mass}"/>
+  	<!-- <inertia ixx="1" ixy="0" ixz="0" iyy="1" iyz="0" izz="1"/> -->
+	<inertia ixx="${base_wheel_mass*base_wheel_radius*base_wheel_radius/4+base_wheel_mass*base_wheel_width*base_wheel_width)}"
+		 ixy="0" ixz="0"
+		 iyy="${base_wheel_mass*base_wheel_radius*base_wheel_radius/4+base_wheel_mass*base_wheel_width*base_wheel_width)}"
+		 iyz="0" izz="${base_wheel_mass*base_wheel_radius*base_wheel_radius/2)}" />
       </inertial>
       <collision>
@@ -281,5 +286,5 @@
   	  <box size="0.025 0.025 0.285"/>
   	</geometry>
-  	w			<material name="grey"/>
+  	<material name="grey"/>
   	<origin rpy="0 0 0" xyz="0 0 0"/>
       </visual>
@@ -1010,6 +1015,9 @@
       <inertial>
   	<origin rpy="0 0 0" xyz="0 0 0"/>
-  	<mass value="1"/>
-  	<inertia ixx="1" ixy="0" ixz="0" iyy="1" iyz="0" izz="1"/>
+  	<mass value="${caster_wheel_mass}"/>
+	<inertia ixx="${caster_wheel_mass*caster_wheel_radius*caster_wheel_radius/4+caster_wheel_mass*caster_wheel_width*caster_wheel_width)}"
+		 ixy="0" ixz="0"
+		 iyy="${caster_wheel_mass*caster_wheel_radius*caster_wheel_radius/4+caster_wheel_mass*caster_wheel_width*caster_wheel_width)}"
+		 iyz="0" izz="${caster_wheel_mass*caster_wheel_radius*caster_wheel_radius/2)}" />
       </inertial>
       <collision>
@@ -1035,6 +1043,9 @@
       <inertial>
   	<origin rpy="0 0 0" xyz="0 0 0"/>
-  	<mass value="1"/>
-  	<inertia ixx="1" ixy="0" ixz="0" iyy="1" iyz="0" izz="1"/>
+  	<mass value="${caster_wheel_mass}"/>
+	<inertia ixx="${caster_wheel_mass*caster_wheel_radius*caster_wheel_radius/4+caster_wheel_mass*caster_wheel_width*caster_wheel_width)}"
+		 ixy="0" ixz="0"
+		 iyy="${caster_wheel_mass*caster_wheel_radius*caster_wheel_radius/4+caster_wheel_mass*caster_wheel_width*caster_wheel_width)}"
+		 iyz="0" izz="${caster_wheel_mass*caster_wheel_radius*caster_wheel_radius/2)}" />
       </inertial>
       <collision>
@@ -1227,4 +1238,5 @@
       <hardwareInterface>EffortJointInterface</hardwareInterface>
       <mechanicalReduction>1</mechanicalReduction>
+      <motorTorqueConstant>20</motorTorqueConstant>
     </actuator>
   </transmission>
@@ -1235,4 +1247,5 @@
       <hardwareInterface>EffortJointInterface</hardwareInterface>
       <mechanicalReduction>1</mechanicalReduction>
+      <motorTorqueConstant>20</motorTorqueConstant>
     </actuator>
   </transmission>
