Commit message: Plow model finished

File: src/redblade_description/urdf/redblade_plow.xacro (robot description, xacro)
@@ -13,7 +13,4 @@
   <xacro:property name="base_wheel_radius" value="0.12" />
   <xacro:property name="base_wheel_mass" value="1.0" />
-  <xacro:property name="caster_wheel_width" value="0.05" />
-  <xacro:property name="caster_wheel_radius" value="0.075" />
-  <xacro:property name="caster_wheel_mass" value="1.0" />
   <xacro:property name="torque" value="20.0" />
   <!-- Import all Gazebo-customization elements, including Gazebo colors -->
@@ -50,21 +47,21 @@
     <origin xyz="0 0 0.195"/>
   </joint>
-    <link name="wheel_left">
-      <visual>
-  	<geometry>
-  	  <cylinder length="0.12" radius="0.1975"/>
-  	</geometry>
-  	<material name="wheel"/>
-  	<origin rpy="1.5707 0 0" xyz="0 0 0"/>
-      </visual>
-      <inertial>
-  	<origin rpy="0 0 0" xyz="0 0 0"/>
-  	<mass value="${base_wheel_mass}"/>
-	<!-- <inertia ixx="1" ixy="0" ixz="0" iyy="1" iyz="0" izz="1"/> -->
-	<inertia ixx="${base_wheel_mass*base_wheel_radius*base_wheel_radius/4+base_wheel_mass*base_wheel_width*base_wheel_width)}"
-		 ixy="0" ixz="0"
-		 iyy="${base_wheel_mass*base_wheel_radius*base_wheel_radius/4+base_wheel_mass*base_wheel_width*base_wheel_width)}"
-		 iyz="0" izz="${base_wheel_mass*base_wheel_radius*base_wheel_radius/2)}" />
-      </inertial>
+  <link name="back_wheel_left">
+    <visual>
+      <geometry>
+	<cylinder length="0.12" radius="0.1975"/>
+      </geometry>
+      <material name="wheel"/>
+      <origin rpy="1.5707 0 0" xyz="0 0 0"/>
+    </visual>
+    <inertial>
+      <origin rpy="0 0 0" xyz="0 0 0"/>
+      <mass value="${base_wheel_mass}"/>
+      <!-- <inertia ixx="1" ixy="0" ixz="0" iyy="1" iyz="0" izz="1"/> -->
+      <inertia ixx="${base_wheel_mass*base_wheel_radius*base_wheel_radius/4+base_wheel_mass*base_wheel_width*base_wheel_width)}"
+	       ixy="0" ixz="0"
+	       iyy="${base_wheel_mass*base_wheel_radius*base_wheel_radius/4+base_wheel_mass*base_wheel_width*base_wheel_width)}"
+	       iyz="0" izz="${base_wheel_mass*base_wheel_radius*base_wheel_radius/2)}" />
+    </inertial>
     <collision>
       <origin rpy="1.5707 0 0" xyz="0 0 0"/>
@@ -73,1074 +70,1152 @@
       </geometry>
     </collision>
-    </link>
-    <joint name="to_wheel_left" type="continuous">
-      <parent link="base_link"/>
-      <child link="wheel_left"/>
-      <axis xyz="0 1 0"/>
-      <origin xyz="0 0.235 0"/>
-    </joint>
-    <link name="wheel_right">
-      <visual>
-  	<geometry>
-  	  <cylinder length="0.12" radius="0.1975"/>
-  	</geometry>
-  	<material name="wheel"/>
-  	<origin rpy="1.5707 0 0" xyz="0 0 0"/>
-      </visual>
-      <inertial>
-  	<origin rpy="0 0 0" xyz="0 0 0"/>
-   	<mass value="${base_wheel_mass}"/>
-  	<!-- <inertia ixx="1" ixy="0" ixz="0" iyy="1" iyz="0" izz="1"/> -->
-	<inertia ixx="${base_wheel_mass*base_wheel_radius*base_wheel_radius/4+base_wheel_mass*base_wheel_width*base_wheel_width)}"
-		 ixy="0" ixz="0"
-		 iyy="${base_wheel_mass*base_wheel_radius*base_wheel_radius/4+base_wheel_mass*base_wheel_width*base_wheel_width)}"
-		 iyz="0" izz="${base_wheel_mass*base_wheel_radius*base_wheel_radius/2)}" />
-      </inertial>
-      <collision>
-	<origin rpy="1.5707 0 0" xyz="0 0 0"/>
-	<geometry>
-	  <cylinder length="0.12" radius="0.1975"/>
-	</geometry>
-      </collision>
-    </link>
-    <joint name="to_wheel_right" type="continuous">
-      <parent link="base_link"/>
-      <child link="wheel_right"/>
-      <axis xyz="0 1 0"/>
-      <origin xyz="0 -0.235 0"/>
-    </joint>
-    <link name="motor_mount_left">
-      <visual>
-  	<geometry>
-  	  <box size="0.025 0.025 0.0575"/>
-  	</geometry>
-  	<material name="grey"/>
-  	<origin rpy="0 0 0" xyz="0 0 0"/>
-      </visual>
-      <inertial>
-  	<origin rpy="0 0 0" xyz="0 0 0"/>
-  	<mass value="1"/>
-  	<inertia ixx="1" ixy="0" ixz="0" iyy="1" iyz="0" izz="1"/>
-      </inertial>
-    </link>
-    <joint name="to_motor_mount_left" type="fixed">
-      <parent link="base_link"/>
-      <child link="motor_mount_left"/>
-      <origin xyz="0 0.14 -0.0412"/>
-    </joint>
-    <link name="motor_mount_right">
-      <visual>
-  	<geometry>
-  	  <box size="0.025 0.025 0.0575"/>
-  	</geometry>
-  	<material name="grey"/>
-  	<origin rpy="0 0 0" xyz="0 0 0"/>
-      </visual>
-      <inertial>
-  	<origin rpy="0 0 0" xyz="0 0 0"/>
-  	<mass value="1"/>
-  	<inertia ixx="1" ixy="0" ixz="0" iyy="1" iyz="0" izz="1"/>
-      </inertial>
-    </link>
-    <joint name="to_motor_mount_right" type="fixed">
-      <parent link="base_link"/>
-      <child link="motor_mount_right"/>
-      <origin xyz="0 -0.14 -0.04125"/>
-    </joint>
-    <link name="motor_area_bottom_left">
-      <visual>
-  	<geometry>
-  	  <box size="0.585 0.025 0.025"/>
-  	</geometry>
-  	<material name="grey"/>
-  	<origin rpy="0 0 0" xyz="0 0 0"/>
-      </visual>
-      <inertial>
-  	<origin rpy="0 0 0" xyz="0 0 0"/>
-  	<mass value="1"/>
-  	<inertia ixx="1" ixy="0" ixz="0" iyy="1" iyz="0" izz="1"/>
-      </inertial>
-    </link>
-    <joint name="to_motor_area_bottom_left" type="fixed">
-      <parent link="motor_mount_left"/>
-      <child link="motor_area_bottom_left"/>
-      <origin xyz="-0.07 0 -0.04125"/>
-    </joint>
-    <link name="motor_area_bottom_right">
-      <visual>
-  	<geometry>
-  	  <box size="0.585 0.025 0.025"/>
-  	</geometry>
-  	<material name="grey"/>
-  	<origin rpy="0 0 0" xyz="0 0 0"/>
-      </visual>
-      <inertial>
-  	<origin rpy="0 0 0" xyz="0 0 0"/>
-  	<mass value="1"/>
-  	<inertia ixx="1" ixy="0" ixz="0" iyy="1" iyz="0" izz="1"/>
-      </inertial>
-    </link>
-    <joint name="to_motor_area_bottom_right" type="fixed">
-      <parent link="motor_mount_right"/>
-      <child link="motor_area_bottom_right"/>
-      <origin xyz="-0.07 0 -0.04125"/>
-    </joint>
-    <link name="motor_area_bottom_front">
-      <visual>
-  	<geometry>
-  	  <box size="0.025 0.255 0.025"/>
-  	</geometry>
-  	<material name="grey"/>
-  	<origin rpy="0 0 0" xyz="0 0 0"/>
-      </visual>
-      <inertial>
-  	<origin rpy="0 0 0" xyz="0 0 0"/>
-  	<mass value="1"/>
-  	<inertia ixx="1" ixy="0" ixz="0" iyy="1" iyz="0" izz="1"/>
-      </inertial>
-    </link>
-    <joint name="to_motor_area_bottom_front" type="fixed">
-      <parent link="motor_area_bottom_left"/>
-      <child link="motor_area_bottom_front"/>
-      <origin xyz="0.28 -0.14 0"/>
-    </joint>
-    <link name="motor_area_bottom_back">
-      <visual>
-  	<geometry>
-  	  <box size="0.025 0.255 0.025"/>
-  	</geometry>
-  	<material name="grey"/>
-  	<origin rpy="0 0 0" xyz="0 0 0"/>
-      </visual>
-      <inertial>
-  	<origin rpy="0 0 0" xyz="0 0 0"/>
-  	<mass value="1"/>
-  	<inertia ixx="1" ixy="0" ixz="0" iyy="1" iyz="0" izz="1"/>
-      </inertial>
-    </link>
-    <joint name="to_motor_area_bottom_back" type="fixed">
-      <parent link="motor_area_bottom_left"/>
-      <child link="motor_area_bottom_back"/>
-      <origin xyz="-0.28 -0.14 0"/>
-    </joint>
-    <link name="motor_area_vent_front_left">
-      <visual>
-  	<geometry>
-  	  <box size="0.025 0.025 0.285"/>
-  	</geometry>
-  	<material name="grey"/>
-  	<origin rpy="0 0 0" xyz="0 0 0"/>
-      </visual>
-      <inertial>
-  	<origin rpy="0 0 0" xyz="0 0 0"/>
-  	<mass value="1"/>
-  	<inertia ixx="1" ixy="0" ixz="0" iyy="1" iyz="0" izz="1"/>
-      </inertial>
-    </link>
-    <joint name="to_motor_area_vent_front_left" type="fixed">
-      <parent link="motor_area_bottom_left"/>
-      <child link="motor_area_vent_front_left"/>
-      <origin xyz="0.28 0 0.155"/>
-    </joint>
-    <link name="motor_area_vent_back_left">
-      <visual>
-  	<geometry>
-  	  <box size="0.025 0.025 0.285"/>
-  	</geometry>
-  	<material name="grey"/>
-  	<origin rpy="0 0 0" xyz="0 0 0"/>
-      </visual>
-      <inertial>
-  	<origin rpy="0 0 0" xyz="0 0 0"/>
-  	<mass value="1"/>
-  	<inertia ixx="1" ixy="0" ixz="0" iyy="1" iyz="0" izz="1"/>
-      </inertial>
-    </link>
-    <joint name="to_motor_area_vent_back_left" type="fixed">
-      <parent link="motor_area_bottom_left"/>
-      <child link="motor_area_vent_back_left"/>
-      <origin xyz="-0.28 0 0.155"/>
-    </joint>
-    <link name="motor_area_vent_front_right">
-      <visual>
-  	<geometry>
-  	  <box size="0.025 0.025 0.285"/>
-  	</geometry>
-  	<material name="grey"/>
-  	<origin rpy="0 0 0" xyz="0 0 0"/>
-      </visual>
-      <inertial>
-  	<origin rpy="0 0 0" xyz="0 0 0"/>
-  	<mass value="1"/>
-  	<inertia ixx="1" ixy="0" ixz="0" iyy="1" iyz="0" izz="1"/>
-      </inertial>
-    </link>
-    <joint name="to_motor_area_vent_front_right" type="fixed">
-      <parent link="motor_area_bottom_right"/>
-      <child link="motor_area_vent_front_right"/>
-      <origin xyz="0.28 0 0.155"/>
-    </joint>
-    <link name="motor_area_vent_back_right">
-      <visual>
-  	<geometry>
-  	  <box size="0.025 0.025 0.285"/>
-  	</geometry>
-  	<material name="grey"/>
-  	<origin rpy="0 0 0" xyz="0 0 0"/>
-      </visual>
-      <inertial>
-  	<origin rpy="0 0 0" xyz="0 0 0"/>
-  	<mass value="1"/>
-  	<inertia ixx="1" ixy="0" ixz="0" iyy="1" iyz="0" izz="1"/>
-      </inertial>
-    </link>
-    <joint name="to_motor_area_vent_back_right" type="fixed">
-      <parent link="motor_area_bottom_right"/>
-      <child link="motor_area_vent_back_right"/>
-      <origin xyz="-0.28 0 0.155"/>
-    </joint>
-    <!-- Motor begin -->
-    <link name="motor_mount_left">
-      <visual>
-  	<geometry>
-  	  <box size="0.025 0.025 0.0575"/>
-  	</geometry>
-  	<material name="grey"/>
-  	<origin rpy="0 0 0" xyz="0 0 0"/>
-      </visual>
-      <inertial>
-  	<origin rpy="0 0 0" xyz="0 0 0"/>
-  	<mass value="1"/>
-  	<inertia ixx="1" ixy="0" ixz="0" iyy="1" iyz="0" izz="1"/>
-      </inertial>
-    </link>
-    <joint name="to_motor_mount_left" type="fixed">
-      <parent link="base_link"/>
-      <child link="motor_mount_left"/>
-      <origin xyz="0 0.14 -0.0412"/>
-    </joint>
-    <link name="motor_mount_right">
-      <visual>
-  	<geometry>
-  	  <box size="0.025 0.025 0.0575"/>
-  	</geometry>
-  	<material name="grey"/>
-  	<origin rpy="0 0 0" xyz="0 0 0"/>
-      </visual>
-      <inertial>
-  	<origin rpy="0 0 0" xyz="0 0 0"/>
-  	<mass value="1"/>
-  	<inertia ixx="1" ixy="0" ixz="0" iyy="1" iyz="0" izz="1"/>
-      </inertial>
-    </link>
-    <joint name="to_motor_mount_right" type="fixed">
-      <parent link="base_link"/>
-      <child link="motor_mount_right"/>
-      <origin xyz="0 -0.14 -0.04125"/>
-    </joint>
-    <link name="motor_area_bottom_left">
-      <visual>
-  	<geometry>
-  	  <box size="0.585 0.025 0.025"/>
-  	</geometry>
-  	<material name="grey"/>
-  	<origin rpy="0 0 0" xyz="0 0 0"/>
-      </visual>
-      <inertial>
-  	<origin rpy="0 0 0" xyz="0 0 0"/>
-  	<mass value="1"/>
-  	<inertia ixx="1" ixy="0" ixz="0" iyy="1" iyz="0" izz="1"/>
-      </inertial>
-    </link>
-    <joint name="to_motor_area_bottom_left" type="fixed">
-      <parent link="motor_mount_left"/>
-      <child link="motor_area_bottom_left"/>
-      <origin xyz="-0.07 0 -0.04125"/>
-    </joint>
-    <link name="motor_area_bottom_right">
-      <visual>
-  	<geometry>
-  	  <box size="0.585 0.025 0.025"/>
-  	</geometry>
-  	<material name="grey"/>
-  	<origin rpy="0 0 0" xyz="0 0 0"/>
-      </visual>
-      <inertial>
-  	<origin rpy="0 0 0" xyz="0 0 0"/>
-  	<mass value="1"/>
-  	<inertia ixx="1" ixy="0" ixz="0" iyy="1" iyz="0" izz="1"/>
-      </inertial>
-    </link>
-    <joint name="to_motor_area_bottom_right" type="fixed">
-      <parent link="motor_mount_right"/>
-      <child link="motor_area_bottom_right"/>
-      <origin xyz="-0.07 0 -0.04125"/>
-    </joint>
-    <link name="motor_area_bottom_front">
-      <visual>
-  	<geometry>
-  	  <box size="0.025 0.255 0.025"/>
-  	</geometry>
-  	<material name="grey"/>
-  	<origin rpy="0 0 0" xyz="0 0 0"/>
-      </visual>
-      <inertial>
-  	<origin rpy="0 0 0" xyz="0 0 0"/>
-  	<mass value="1"/>
-  	<inertia ixx="1" ixy="0" ixz="0" iyy="1" iyz="0" izz="1"/>
-      </inertial>
-    </link>
-    <joint name="to_motor_area_bottom_front" type="fixed">
-      <parent link="motor_area_bottom_left"/>
-      <child link="motor_area_bottom_front"/>
-      <origin xyz="0.28 -0.14 0"/>
-    </joint>
-    <link name="motor_area_bottom_back">
-      <visual>
-  	<geometry>
-  	  <box size="0.025 0.255 0.025"/>
-  	</geometry>
-  	<material name="grey"/>
-  	<origin rpy="0 0 0" xyz="0 0 0"/>
-      </visual>
-      <inertial>
-  	<origin rpy="0 0 0" xyz="0 0 0"/>
-  	<mass value="1"/>
-  	<inertia ixx="1" ixy="0" ixz="0" iyy="1" iyz="0" izz="1"/>
-      </inertial>
-    </link>
-    <joint name="to_motor_area_bottom_back" type="fixed">
-      <parent link="motor_area_bottom_left"/>
-      <child link="motor_area_bottom_back"/>
-      <origin xyz="-0.28 -0.14 0"/>
-    </joint>
-    <link name="motor_area_vent_front_left">
-      <visual>
-  	<geometry>
-  	  <box size="0.025 0.025 0.285"/>
-  	</geometry>
-  	<material name="grey"/>
-  	<origin rpy="0 0 0" xyz="0 0 0"/>
-      </visual>
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
Commit message: Adding in working skid steer drive

File: src/redblade_description/urdf/redblade_plow.xacro (robot description, xacro)
@@ -270,5 +270,5 @@
       <origin rpy="0 0 0" xyz="0 0 0"/>
       <mass value="1"/>
-      <inertia ixx="1" ixy="0" ixz="0" iyy="1" iyz="0" izz="1"/>
+     <inertia ixx="1" ixy="0" ixz="0" iyy="1" iyz="0" izz="1"/>
     </inertial>
   </link>
@@ -1233,3 +1233,21 @@
     </actuator>
   </transmission>
+  <transmission name="front_wheel_left_tran">
+    <type>transmission_interface/SimpleTransmission</type>
+    <joint name="to_front_wheel_left"/>
+    <actuator name="motor3">
+      <hardwareInterface>EffortJointInterface</hardwareInterface>
+      <mechanicalReduction>1</mechanicalReduction>
+      <motorTorqueConstant>20</motorTorqueConstant>
+    </actuator>
+  </transmission>
+  <transmission name="front_wheel_right_tran">
+    <type>transmission_interface/SimpleTransmission</type>
+    <joint name="to_front_wheel_right"/>
+    <actuator name="motor4">
+      <hardwareInterface>EffortJointInterface</hardwareInterface>
+      <mechanicalReduction>1</mechanicalReduction>
+      <motorTorqueConstant>20</motorTorqueConstant>
+    </actuator>
+  </transmission>
 </robot>
