Commit message: Publishing redblade odometry in gazebo

File: src/redblade_description/urdf/redblade.urdf (robot description, URDF)
Before this commit: robot redblade, 62 links, 61 joints
Links:
- removed link caster_left
- removed link caster_right
- removed link deck_area_bottom_left
- removed link deck_area_bottom_right
- removed link deck_area_bottom_side_left
- removed link deck_area_bottom_side_right
- removed link deck_area_vent_back_left
- removed link deck_area_vent_back_right
- removed link deck_area_vent_front_left
- removed link deck_area_vent_front_right
- removed link laser
- removed link lidar_area_bottom
- removed link lidar_area_vert_left
- removed link lidar_area_vert_right
- removed link motor_mount_left
- removed link motor_mount_right
- removed link wheel_left
- removed link wheel_right
- added link back_motor_mount_left, mass 1; visual box size=0.025 0.025 0.0575
- added link back_motor_mount_right, mass 1; visual box size=0.025 0.025 0.0575
- added link back_wheel_left, mass 1.0; collision cylinder length=0.12 radius=0.1975; visual cylinder length=0.12 radius=0.1975
- added link back_wheel_right, mass 1.0; collision cylinder length=0.12 radius=0.1975; visual cylinder length=0.12 radius=0.1975
- added link front_link, mass 1; visual box size=0.025 0.35 0.025
- added link front_motor_area_bottom_back, mass 1; visual box size=0.025 0.255 0.025
- added link front_motor_area_bottom_front, mass 1; visual box size=0.025 0.255 0.025
- added link front_motor_area_bottom_left, mass 1; visual box size=0.585 0.025 0.025
- added link front_motor_area_bottom_right, mass 1; visual box size=0.585 0.025 0.025
- added link front_motor_area_vent_back_left, mass 1; visual box size=0.025 0.025 0.285
- added link front_motor_area_vent_back_right, mass 1; visual box size=0.025 0.025 0.285
- added link front_motor_area_vent_front_left, mass 1; visual box size=0.025 0.025 0.285
- added link front_motor_area_vent_front_right, mass 1; visual box size=0.025 0.025 0.285
- added link front_motor_mount_left, mass 1; visual box size=0.025 0.025 0.0575
- added link front_motor_mount_right, mass 1; visual box size=0.025 0.025 0.0575
- added link front_wheel_left, mass 1.0; collision cylinder length=0.12 radius=0.1975; visual cylinder length=0.12 radius=0.1975
- added link front_wheel_right, mass 1.0; collision cylinder length=0.12 radius=0.1975; visual cylinder length=0.12 radius=0.1975
- link base_footprint: mass 1 -> None
- link base_link: geometry visual box size=0.025 0.35 0.025
Joints:
- removed joint to_caster_left
- removed joint to_caster_right
- removed joint to_deck_area_bottom_left
- removed joint to_deck_area_bottom_right
- removed joint to_deck_area_bottom_side_left
- removed joint to_deck_area_bottom_side_right
- removed joint to_deck_area_vent_back_left
- removed joint to_deck_area_vent_back_right
- removed joint to_deck_area_vent_front_left
- removed joint to_deck_area_vent_front_right
- removed joint to_laser
- removed joint to_lidar_area_bottom
- removed joint to_lidar_area_vert_left
- removed joint to_lidar_area_vert_right
- removed joint to_motor_mount_left
- removed joint to_motor_mount_right
- removed joint to_wheel_left
- removed joint to_wheel_right
- added joint to_back_motor_mount_left: type fixed, parent base_link, child back_motor_mount_left, origin xyz=0 0.14 -0.0412
- added joint to_back_motor_mount_right: type fixed, parent base_link, child back_motor_mount_right, origin xyz=0 -0.14 -0.04125
- added joint to_back_wheel_left: type continuous, parent base_link, child back_wheel_left, origin xyz=0 0.235 0, axis 0 1 0
- added joint to_back_wheel_right: type continuous, parent base_link, child back_wheel_right, origin xyz=0 -0.235 0, axis 0 1 0
- added joint to_front_link: type fixed, parent front_motor_area_bottom_left, child front_link, origin xyz=-0.07 -0.14 0.0825
- added joint to_front_motor_area_bottom_back: type fixed, parent front_motor_area_bottom_left, child front_motor_area_bottom_back, origin xyz=-0.28 -0.14 0
- added joint to_front_motor_area_bottom_front: type fixed, parent front_motor_area_bottom_left, child front_motor_area_bottom_front, origin xyz=0.28 -0.14 0
- added joint to_front_motor_area_bottom_left: type fixed, parent front_motor_area_vent_front_left, child front_motor_area_bottom_left, origin xyz=-0.28 0 -0.155
- added joint to_front_motor_area_bottom_right: type fixed, parent front_motor_area_vent_front_right, child front_motor_area_bottom_right, origin xyz=-0.28 0 -0.155
- added joint to_front_motor_area_vent_back_left: type fixed, parent main_area_bottom_front, child front_motor_area_vent_back_left, origin xyz=-0.56 0.14 -0.155
- added joint to_front_motor_area_vent_back_right: type fixed, parent main_area_bottom_front, child front_motor_area_vent_back_right, origin xyz=-0.56 -0.14 -0.155
- added joint to_front_motor_area_vent_front_left: type fixed, parent main_area_bottom_front, child front_motor_area_vent_front_left, origin xyz=0 0.14 -0.155
- added joint to_front_motor_area_vent_front_right: type fixed, parent main_area_bottom_front, child front_motor_area_vent_front_right, origin xyz=0 -0.14 -0.155
- added joint to_front_motor_mount_left: type fixed, parent front_motor_area_bottom_left, child front_motor_mount_left, origin xyz=-0.07 0 0.0412
- added joint to_front_motor_mount_right: type fixed, parent front_motor_area_bottom_right, child front_motor_mount_right, origin xyz=-0.07 0 0.0412
- added joint to_front_wheel_left: type continuous, parent front_link, child front_wheel_left, origin xyz=0 0.235 0, axis 0 1 0
- added joint to_front_wheel_right: type continuous, parent front_link, child front_wheel_right, origin xyz=0 -0.235 0, axis 0 1 0
- joint to_motor_area_bottom_left: parent motor_mount_left -> back_motor_mount_left
- joint to_motor_area_bottom_right: parent motor_mount_right -> back_motor_mount_right
